Commit message: saving urdf changes

File: lerobot/configs/giraffe.urdf (robot description, URDF)
Before this commit: robot giraffe, 7 links, 6 joints
Joints:
- joint base_link_shoulder_pan_joint: axis -4.930380657631324e-32 2.37251531204244e-15 1.0 -> -4.930380657631324e-32 2.37251531204244e-15 -1.0
- joint elbow_wrist_1_joint: axis -0.9999998631005341 -1.23112379231774e-10 0.0007583461697307804 -> 0.9999998631005341 1.23112379231774e-10 -0.0007583461697307804
- joint shoulder_lift_elbow_joint: axis 1.0000002880403989 -1.245357002578147e-10 -3.456292375562768e-07 -> -1.0000002880403989 1.245357002578147e-10 3.456292375562768e-07
- joint shoulder_pan_shoulder_lift_joint: limit lower=-0.785398 upper=1.658063 effort=1000000 velocity=1000000 -> lower=0.0 upper=2.18166 effort=1000000 velocity=1000000
- joint wrist_1_wrist_2_joint: axis -0.9999449329225374 0.006662002215913354 -0.008132268196377131 -> 0.9999449329225374 -0.006662002215913354 0.008132268196377131

Commit message: added new urdf with fixed joint origins and base origin

File: lerobot/configs/giraffe.urdf (robot description, URDF)
Before this commit: robot giraffe, 7 links, 6 joints
Links:
- link base_link: mass 0.8122108919622869 -> 0.812210891962288; geometry collision mesh filename=meshes/base_link.stl scale=0.001 0.001 0.001; visual mesh filename=meshes/base_link.stl scale=0.001 0.001 0.001
- link elbow: mass 0.3407348467366932 -> 0.34073484673669374; geometry collision mesh filename=meshes/elbow.stl scale=0.001 0.001 0.001; visual mesh filename=meshes/elbow.stl scale=0.001 0.001 0.001
- link gripper: mass 0.12794799500230522 -> 0.12794799500230405; geometry collision mesh filename=meshes/gripper.stl scale=0.001 0.001 0.001; visual mesh filename=meshes/gripper.stl scale=0.001 0.001 0.001
- link shoulder_lift: mass 0.34405090664671173 -> 0.34405090664671145; geometry collision mesh filename=meshes/shoulder_lift.stl scale=0.001 0.001 0.001; visual mesh filename=meshes/shoulder_lift.stl scale=0.001 0.001 0.001
- link shoulder_pan: mass 0.2502336197461597 -> 0.25023361974615993; geometry collision mesh filename=meshes/shoulder_pan.stl scale=0.001 0.001 0.001; visual mesh filename=meshes/shoulder_pan.stl scale=0.001 0.001 0.001
- link wrist_1: mass 0.11585466541730399 -> 0.11585466541730426; geometry collision mesh filename=meshes/wrist_1.stl scale=0.001 0.001 0.001; visual mesh filename=meshes/wrist_1.stl scale=0.001 0.001 0.001
- link wrist_2: mass 0.20479740953235442 -> 0.20479740953235626; geometry collision mesh filename=meshes/wrist_2.stl scale=0.001 0.001 0.001; visual mesh filename=meshes/wrist_2.stl scale=0.001 0.001 0.001
Joints:
- joint base_link_shoulder_pan_joint: axis -4.930380657631324e-32 2.37251531204244e-15 -1.0 -> 1.0000000000000002e-06 -0.0007589999999976223 1.0000000000000002; limit lower=-1.832596 upper=1.832596 effort=1000000 velocity=1000000 -> lower=-1.570796 upper=1.570796 effort=1000000 velocity=1000000; origin xyz=0.09891995753862716 -0.00013303607482287617 0.05455000000000001 rpy=3.189786117866041e-15 3.393805650568627e-16 -0.0007586542251351899 -> xyz=0.0024422199571167862 -2.1995292539264472e-05 0.017300000259741807 rpy=3.140833999582909 5.755561299100456e-07 -2.1828320944785756e-10
- joint elbow_wrist_1_joint: axis 0.9999998631005341 1.23112379231774e-10 -0.0007583461697307804 -> -0.9999998631005341 -1.23112379231774e-10 0.0007583461697307803; limit lower=-1.797689 upper=1.797689 effort=1000000 velocity=1000000 -> lower=-1.570796 upper=1.570796 effort=1000000 velocity=1000000; origin xyz=-0.03761630670794674 -0.0022157899953267803 0.12026017684096592 rpy=1.8787933722333255e-13 2.512616851854867e-14 -2.476481313343611e-10 -> xyz=-0.0004656960202010452 0.0022157899999533637 -0.12026018130602735 rpy=-3.1415926535896053 -3.2273446080007626e-14 2.476481313354115e-10
- joint shoulder_lift_elbow_joint: axis -1.0000002880403989 1.245357002578147e-10 3.456292375562768e-07 -> -1.000000288040399 -1.245357002589312e-10 -3.4562924470333753e-07; limit lower=-1.53589 upper=1.780236 effort=1000000 velocity=1000000 -> lower=0.0 upper=3.141593 effort=1000000 velocity=1000000; origin xyz=0.037893485547286214 0.10949145999216181 -0.025196435301140276 rpy=3.1415926535895418 2.265006756586156e-14 -3.364010369466755e-10 -> xyz=-0.03680651674664366 0.02516801999240762 0.10949145809248002 rpy=3.1415926535895418 -3.694418900791044e-14 3.312801036937707e-10
- joint shoulder_pan_shoulder_lift_joint: axis -0.9999997122218972 2.0674449874803995e-10 0.0007586541523615138 -> 0.9999992880405297 0.0007590002067442921 -3.4638786203060774e-07; limit lower=0.0 upper=2.18166 effort=1000000 velocity=1000000 -> lower=0.0 upper=1.570796 effort=1000000 velocity=1000000; origin xyz=0.02571940999999997 0.018944660000000037 0.017376069999999952 rpy=1.5707963267950535 -2.0674681179012968e-10 -1.5715549810200329 -> xyz=0.02570547999999961 0.018366289999999865 -0.05461217000000003 rpy=1.5707963267950535 2.0674681721032812e-10 1.57155498102004
- joint wrist_1_wrist_2_joint: axis 0.9999449329225374 -0.006662002215913354 0.008132268196377131 -> -0.9999449329225374 0.006662002215913354 -0.008132268196377131; origin xyz=0.027165827341760113 -0.00019891999664992 0.06031796682590525 rpy=-3.049102007927164 1.5625820319968764 -1.4783560893203032 -> xyz=0.02716582734176012 -0.0001989299966499214 0.06031796682590525 rpy=-3.049102007927164 1.5625820319968764 -1.478356089320303
- joint wrist_2_gripper_joint: axis -0.007420635544791429 -0.0007590000001611277 -0.9999726580742655 -> -0.007420635544791429 -0.0007590000001611273 -0.9999726580742653; origin xyz=-0.017171676526959914 -0.019310353391698003 -0.025579471562416883 rpy=-1.5708498378135036 -0.0081791843801793 0.0007586796016244804 -> xyz=-0.017171676526959844 -0.019310353391698006 -0.025579471562416866 rpy=-1.5708498378135036 -0.0081791843801793 0.0007586796016247202

Commit message: updated urdf origins again

File: lerobot/configs/giraffe.urdf (robot description, URDF)
Before this commit: robot giraffe, 7 links, 6 joints
Links:
- link base_link: mass 0.812210891962288 -> 0.8122108919622884
Joints:
- joint base_link_shoulder_pan_joint: axis 1.0000000000000002e-06 -0.0007589999999976223 1.0000000000000002 -> 1e-06 -0.000758999999997622 1.0; origin xyz=0.0024422199571167862 -2.1995292539264472e-05 0.017300000259741807 rpy=3.140833999582909 5.755561299100456e-07 -2.1828320944785756e-10 -> xyz=-7.78471460176888e-06 -2.200004287780052e-05 0.017299999085318825 rpy=3.140833999582908 5.755561288912283e-07 1.5707963265766136
- joint elbow_wrist_1_joint: axis -0.9999998631005341 -1.23112379231774e-10 0.0007583461697307803 -> 0.000758346169637338 0.0007590000001867616 0.999999863100534; origin xyz=-0.0004656960202010452 0.0022157899999533637 -0.12026018130602735 rpy=-3.1415926535896053 -3.2273446080007626e-14 2.476481313354115e-10 -> xyz=0.12026183003074924 0.002124210014976935 -0.00046737727122078134 rpy=-3.1415926535896053 -3.2273229239573103e-14 2.4764813144400373e-10
- joint shoulder_lift_elbow_joint: axis -1.000000288040399 -1.245357002589312e-10 -3.4562924470333753e-07 -> -6.536117188437661e-07 -0.000758999999905602 -0.9999992872820326; origin xyz=-0.03680651674664366 0.02516801999240762 0.10949145809248002 rpy=3.1415926535895418 -3.694418900791044e-14 3.312801036937707e-10 -> xyz=0.10947230258306867 0.025279000022638557 0.03678740220353282 rpy=3.1415926535895418 -3.694418900791045e-14 3.312801036938606e-10
- joint shoulder_pan_shoulder_lift_joint: axis 0.9999992880405297 0.0007590002067442921 -3.4638786203060774e-07 -> -3.456292077591485e-07 -1.5691907467237958e-13 -1.0000002880403989; origin xyz=0.02570547999999961 0.018366289999999865 -0.05461217000000003 rpy=1.5707963267950535 2.0674681721032812e-10 1.57155498102004 -> xyz=-0.018324870000000392 0.025746959999999867 -0.054606550000000066 rpy=1.5707963267950535 2.067468172103282e-10 1.57155498102004
- joint wrist_1_wrist_2_joint: axis -0.9999449329225374 0.006662002215913354 -0.008132268196377131 -> -0.006668805523688299 -0.999976960468889 0.0008047864868520909; origin xyz=0.02716582734176012 -0.0001989299966499214 0.06031796682590525 rpy=-3.049102007927164 1.5625820319968764 -1.478356089320303 -> xyz=0.0603181067045017 -0.00017376999257662896 -0.02716566723557007 rpy=-3.049102007927164 1.5625820319968764 -1.4783560893203032
- joint wrist_2_gripper_joint: axis -0.007420635544791429 -0.0007590000001611273 -0.9999726580742653 -> 0.9999726580742655 -6.000000001073452e-06 -0.007420635544791427; origin xyz=-0.017171676526959844 -0.019310353391698006 -0.025579471562416866 rpy=-1.5708498378135036 -0.0081791843801793 0.0007586796016247202 -> xyz=0.019497289303155634 -0.01740085346148174 -0.025281061620179096 rpy=-1.5708498378135036 -0.008179184380179302 0.00075867960162472
